Commit message: feat: Update robot with camera, lidar and wheels

File: src/my_robot/urdf/my_robot.xacro (robot description, xacro)
@@ -1,11 +1,11 @@
-<?xml version='1.0'?>
+<?xml version="1.0"?>
 <robot name="my_robot" xmlns:xacro="http://www.ros.org/wiki/xacro">
-  <link name="robot_footprint"></link>
+  <link name="robot_footprint"/>
   <joint name="robot_footprint_joint" type="fixed">
-    <origin xyz="0 0 0" rpy="0 0 0" />
+    <origin xyz="0 0 0" rpy="0 0 0"/>
     <parent link="robot_footprint"/>
-    <child link="chassis" />
+    <child link="chassis"/>
   </joint>
-  <link name='chassis'>
+  <link name="chassis">
     <pose>0 0 0.1 0 0 0</pose>
     <inertial>
@@ -18,5 +18,5 @@
       />
     </inertial>
-    <collision name='collision'>
+    <collision name="collision">
       <origin xyz="0 0 0" rpy=" 0 0 0"/>
       <geometry>
@@ -24,5 +24,5 @@
       </geometry>
     </collision>
-    <visual name='chassis_visual'>
+    <visual name="chassis_visual">
       <origin xyz="0 0 0" rpy=" 0 0 0"/>
       <geometry>
@@ -30,5 +30,5 @@
       </geometry>
     </visual>
-    <collision name='back_caster_collision'>
+    <collision name="back_caster_collision">
       <origin xyz="-0.15 0 -0.05" rpy=" 0 0 0"/>
       <geometry>
@@ -36,5 +36,5 @@
       </geometry>
     </collision>
-    <visual name='back_caster_visual'>
+    <visual name="back_caster_visual">
       <origin xyz="-0.15 0 -0.05" rpy=" 0 0 0"/>
       <geometry>
@@ -42,5 +42,5 @@
       </geometry>
     </visual>
-    <collision name='front_caster_collision'>
+    <collision name="front_caster_collision">
       <origin xyz="0.15 0 -0.05" rpy=" 0 0 0"/>
       <geometry>
@@ -48,5 +48,5 @@
       </geometry>
     </collision>
-    <visual name='front_caster_visual'>
+    <visual name="front_caster_visual">
       <origin xyz="0.15 0 -0.05" rpy=" 0 0 0"/>
       <geometry>
@@ -55,3 +55,131 @@
     </visual>
   </link>
+  <link name="left-wheel">
+    <pose>0 0 0 0 0 0</pose>
+    <inertial>
+      <mass value="5.0"/>
+      <origin xyz="0.0 0 0" rpy=" 0 1.5707 1.5707"/>
+      <inertia
+          ixx="0.1" ixy="0" ixz="0"
+          iyy="0.1" iyz="0"
+          izz="0.1"
+      />
+    </inertial>
+    <collision name="collision">
+      <origin xyz="0 0 0" rpy=" 0 1.5707 1.5707"/>
+      <geometry>
+        <cylinder radius="0.1" length="0.05"/>
+      </geometry>
+    </collision>
+    <visual name="left_wheel_visual">
+      <origin xyz="0 0 0" rpy=" 0 1.5707 1.5707"/>
+      <geometry>
+        <cylinder radius="0.1" length="0.05"/>
+      </geometry>
+    </visual>
+  </link>
+  <link name="right_wheel">
+    <pose>0 0 0 0 0 0</pose>
+    <inertial>
+      <mass value="5.0"/>
+      <origin xyz="0.0 0 0" rpy=" 0 1.5707 1.5707"/>
+      <inertia
+          ixx="0.1" ixy="0" ixz="0"
+          iyy="0.1" iyz="0"
+          izz="0.1"
+      />
+    </inertial>
+    <collision name="collision">
+      <origin xyz="0 0 0" rpy=" 0 1.5707 1.5707"/>
+      <geometry>
+        <cylinder radius="0.1" length="0.05"/>
+      </geometry>
+    </collision>
+    <visual name="right_wheel_visual">
+      <origin xyz="0 0 0" rpy=" 0 1.5707 1.5707"/>
+      <geometry>
+        <cylinder radius="0.1" length="0.05"/>
+      </geometry>
+    </visual>
+  </link>
+  <joint type="continuous" name="left_wheel_hinge">
+    <origin xyz="0 0.15 0" rpy="0 0 0"/>
+    <child link="left_wheel"/>
+    <parent link="chassis"/>
+    <axis xyz="0 1 0" rpy="0 0 0"/>
+    <limit effort="10000" velocity="1000"/>
+    <dynamics damping="1.0" friction="1.0"/>
+  </joint>
+  <joint type="continuous" name="right_wheel_hinge">
+    <origin xyz="0 -0.15 0" rpy="0 0 0"/>
+    <child link="right_wheel"/>
+    <parent link="chassis"/>
+    <axis xyz="0 1 0" rpy="0 0 0"/>
+    <limit effort="10000" velocity="1000"/>
+    <dynamics damping="1.0" friction="1.0"/>
+  </joint>
+  <link name="camera">
+    <pose>0 0 0 0 0 0</pose>
+    <inertial>
+      <mass value="0.1"/>
+      <origin xyz="0.0 0 0" rpy="0.0 0 0"/>
+      <inertia
+          ixx="1e-6" ixy="0" ixz="0"
+          iyy="1e-6" iyz="0"
+          izz="1e-6"
+      />
+    </inertial>
+    <collision name="collision">
+      <origin xyz="0 0 0" rpy=" 0 0 0"/>
+      <geometry>
+        <box size="0.05 0.05 0.05"/>
+      </geometry>
+    </collision>
+    <visual name="camera_visual">
+      <origin xyz="0 0 0" rpy="0 0 0"/>
+      <geometry>
+        <box size="0.05 0.05 0.05"/>
+      </geometry>
+    </visual>
+  </link>
+  <joint type="fixed" name="camera_joint">
+    <origin xyz="0.2 0 0" rpy="0 0 0"/>
+    <child link="camera"/>
+    <parent link="chassis"/>
+    <axis xyz="0 1 0" rpy="0 0 0"/>
+    <limit effort="10000" velocity="1000"/>
+    <dynamics damping="1.0" friction="1.0"/>
+  </joint>
+  <link name="hokuyo">
+    <pose>0 0 0 0 0 0</pose>
+    <inertial>
+      <mass value="1e-5"/>
+      <origin xyz="0.0 0 0" rpy="0.0 0 0"/>
+      <inertia
+          ixx="1e-6" ixy="0" ixz="0"
+          iyy="1e-6" iyz="0"
+          izz="1e-6"
+      />
+    </inertial>
+    <collision name="collision">
+      <origin xyz="0 0 0" rpy=" 0 0 0"/>
+      <geometry>
+        <box size="0.1 0.1 0.1"/>
+      </geometry>
+    </collision>
+    <visual name="hokuyo_visual">
+      <origin xyz="0 0 0" rpy="0 0 0"/>
+      <geometry>
+        <mesh filename="package://my_robot/meshes/hokuyo.dae"/>
+      </geometry>
+    </visual>
+  </link>
+  <joint type="fixed" name="hokuyo_joint">
+    <origin xyz="0.15 0.0 0.1" rpy="0 0 0"/>
+    <child link="hokuyo"/>
+    <parent link="chassis"/>
+    <axis xyz="0 1 0" rpy="0 0 0"/>
+    <limit effort="10000" velocity="1000"/>
+    <dynamics damping="1.0" friction="1.0"/>
+  </joint>
 </robot>

Commit message: fix: Ammend left wheel link

File: src/my_robot/urdf/my_robot.xacro (robot description, xacro)
@@ -56,5 +56,5 @@
     </visual>
   </link>
-  <link name="left-wheel">
+  <link name="left_wheel">
     <pose>0 0 0 0 0 0</pose>
     <inertial>

Commit message: feat: Update robot

File: src/my_robot/urdf/my_robot.xacro (robot description, xacro)
@@ -1,6 +1,6 @@
-<?xml version="1.0"?>
+<?xml version='1.0'?>
 <robot name="my_robot" xmlns:xacro="http://www.ros.org/wiki/xacro">
-  <link name="robot_footprint"/>
-  <xacro:include filename="$(find my_robot)/urdf/my_robot.gazebo" />
+  <link name="robot_footprint"></link>
+  <xacro:include filename="$(find my_robot)/urdf/my_robot.gazebo"/>
   <joint name="robot_footprint_joint" type="fixed">
     <origin xyz="0 0 0" rpy="0 0 0"/>
@@ -8,8 +8,8 @@
     <child link="chassis"/>
   </joint>
-  <link name="chassis">
+  <link name='chassis'>
     <pose>0 0 0.1 0 0 0</pose>
     <inertial>
-      <mass value="15.0"/>
+      <mass value="10.0"/>
       <origin xyz="0.0 0 0" rpy=" 0 0 0"/>
       <inertia
@@ -19,42 +19,102 @@
       />
     </inertial>
-    <collision name="collision">
+    <collision name='chassis_collision'>
       <origin xyz="0 0 0" rpy=" 0 0 0"/>
       <geometry>
-        <box size=".4 .2 .1"/>
-      </geometry>
-    </collision>
-    <visual name="chassis_visual">
+        <box size="2. .9 .1"/>
+      </geometry>
+    </collision>
+    <visual name='chassis_visual'>
       <origin xyz="0 0 0" rpy=" 0 0 0"/>
       <geometry>
-        <box size=".4 .2 .1"/>
-      </geometry>
-    </visual>
-    <collision name="back_caster_collision">
-      <origin xyz="-0.15 0 -0.05" rpy=" 0 0 0"/>
-      <geometry>
-        <sphere radius="0.0499"/>
-      </geometry>
-    </collision>
-    <visual name="back_caster_visual">
-      <origin xyz="-0.15 0 -0.05" rpy=" 0 0 0"/>
-      <geometry>
-        <sphere radius="0.05"/>
-      </geometry>
-    </visual>
-    <collision name="front_caster_collision">
-      <origin xyz="0.15 0 -0.05" rpy=" 0 0 0"/>
-      <geometry>
-        <sphere radius="0.0499"/>
-      </geometry>
-    </collision>
-    <visual name="front_caster_visual">
-      <origin xyz="0.15 0 -0.05" rpy=" 0 0 0"/>
-      <geometry>
-        <sphere radius="0.05"/>
-      </geometry>
-    </visual>
-  </link>
-  <link name="left_wheel">
+        <box size="2. .9 .1"/>
+      </geometry>
+    </visual>
+    <collision name='sensor_platform_collision'>
+      <origin xyz="0.8 0 0.1" rpy=" 0 0 0"/>
+      <geometry>
+        <box size=".1 .1 .3"/>
+      </geometry>
+    </collision>
+    <visual name='sensor_platform_visual'>
+      <origin xyz="0.8 0 0.1" rpy=" 0 0 0"/>
+      <geometry>
+        <box size=".1 .1 .3"/>
+      </geometry>
+    </visual>
+    <collision name='front_left_caster_collision'>
+      <origin xyz="0.9 .35 -0.05" rpy=" 0 0 0"/>
+      <geometry>
+        <sphere radius="0.0499"/>
+      </geometry>
+    </collision>
+    <visual name='front_left_caster_visual'>
+      <origin xyz="0.9 .35 -0.05" rpy=" 0 0 0"/>
+      <geometry>
+        <sphere radius="0.05"/>
+      </geometry>
+    </visual>
+    <collision name='front_right_caster_collision'>
+      <origin xyz="0.9 -0.35 -0.05" rpy=" 0 0 0"/>
+      <geometry>
+        <sphere radius="0.0499"/>
+      </geometry>
+    </collision>
+    <visual name='front_right_caster_visual'>
+      <origin xyz="0.9 -0.35 -0.05" rpy=" 0 0 0"/>
+      <geometry>
+        <sphere radius="0.05"/>
+      </geometry>
+    </visual>
+    <collision name='center_left_caster_collision'>
+      <origin xyz="0 0.35 -0.05" rpy=" 0 0 0"/>
+      <geometry>
+        <sphere radius="0.0499"/>
+      </geometry>
+    </collision>
+    <visual name='center_left_caster_visual'>
+      <origin xyz="0 0.35 -0.05" rpy=" 0 0 0"/>
+      <geometry>
+        <sphere radius="0.05"/>
+      </geometry>
+    </visual>
+    <collision name='center_right_caster_collision'>
+      <origin xyz="0 -0.35 -0.05" rpy=" 0 0 0"/>
+      <geometry>
+        <sphere radius="0.0499"/>
+      </geometry>
+    </collision>
+    <visual name='center_right_caster_visual'>
+      <origin xyz="0 -0.35 -0.05" rpy=" 0 0 0"/>
+      <geometry>
+        <sphere radius="0.05"/>
+      </geometry>
+    </visual>
+    <collision name='rear_left_caster_collision'>
+      <origin xyz="-0.9 0.35 -0.05" rpy=" 0 0 0"/>
+      <geometry>
+        <sphere radius="0.0499"/>
+      </geometry>
+    </collision>
+    <visual name='rear_left_caster_visual'>
+      <origin xyz="-0.9 0.35 -0.05" rpy=" 0 0 0"/>
+      <geometry>
+        <sphere radius="0.05"/>
+      </geometry>
+    </visual>
+    <collision name='rear_right_caster_collision'>
+      <origin xyz="-0.9 -0.35 -0.05" rpy=" 0 0 0"/>
+      <geometry>
+        <sphere radius="0.0499"/>
+      </geometry>
+    </collision>
+    <visual name='rear_right_caster_visual'>
+      <origin xyz="-0.9 -0.35 -0.05" rpy=" 0 0 0"/>
+      <geometry>
+        <sphere radius="0.05"/>
+      </geometry>
+    </visual>
+  </link>
+  <link name='front_left_wheel'>
     <pose>0 0 0 0 0 0</pose>
     <inertial>
@@ -67,18 +127,18 @@
       />
     </inertial>
-    <collision name="collision">
-      <origin xyz="0 0 0" rpy=" 0 1.5707 1.5707"/>
-      <geometry>
-        <cylinder radius="0.1" length="0.05"/>
-      </geometry>
-    </collision>
-    <visual name="left_wheel_visual">
-      <origin xyz="0 0 0" rpy=" 0 1.5707 1.5707"/>
-      <geometry>
-        <cylinder radius="0.1" length="0.05"/>
-      </geometry>
-    </visual>
-  </link>
-  <link name="right_wheel">
+    <collision name='front_left_wheel_collision'>
+      <origin xyz="0 0 0" rpy=" 0 1.5707 1.5707"/>
+      <geometry>
+        <cylinder radius="0.14" length="0.21"/>
+      </geometry>
+    </collision>
+    <visual name='front_left_wheel_visual'>
+      <origin xyz="0 0 0" rpy=" 0 1.5707 1.5707"/>
+      <geometry>
+        <cylinder radius="0.14" length="0.21"/>
+      </geometry>
+    </visual>
+  </link>
+  <link name='front_right_wheel'>
     <pose>0 0 0 0 0 0</pose>
     <inertial>
@@ -91,34 +151,98 @@
       />
     </inertial>
-    <collision name="collision">
-      <origin xyz="0 0 0" rpy=" 0 1.5707 1.5707"/>
-      <geometry>
-        <cylinder radius="0.1" length="0.05"/>
-      </geometry>
-    </collision>
-    <visual name="right_wheel_visual">
-      <origin xyz="0 0 0" rpy=" 0 1.5707 1.5707"/>
-      <geometry>
-        <cylinder radius="0.1" length="0.05"/>
-      </geometry>
-    </visual>
-  </link>
-  <joint type="continuous" name="left_wheel_hinge">
-    <origin xyz="0 0.15 0" rpy="0 0 0"/>
-    <child link="left_wheel"/>
-    <parent link="chassis"/>
-    <axis xyz="0 1 0" rpy="0 0 0"/>
-    <limit effort="10000" velocity="1000"/>
-    <dynamics damping="1.0" friction="1.0"/>
-  </joint>
-  <joint type="continuous" name="right_wheel_hinge">
-    <origin xyz="0 -0.15 0" rpy="0 0 0"/>
-    <child link="right_wheel"/>
-    <parent link="chassis"/>
-    <axis xyz="0 1 0" rpy="0 0 0"/>
-    <limit effort="10000" velocity="1000"/>
-    <dynamics damping="1.0" friction="1.0"/>
-  </joint>
-  <link name="camera">
+    <collision name='front_right_wheel_collision'>
+      <origin xyz="0 0 0" rpy=" 0 1.5707 1.5707"/>
+      <geometry>
+        <cylinder radius="0.14" length="0.21"/>
+      </geometry>
+    </collision>
+    <visual name='front_right_wheel_visual'>
+      <origin xyz="0 0 0" rpy=" 0 1.5707 1.5707"/>
+      <geometry>
+        <cylinder radius="0.14" length="0.21"/>
+      </geometry>
+    </visual>
+  </link>
+  <link name='rear_left_wheel'>
+    <pose>0 0 0 0 0 0</pose>
+    <inertial>
+      <mass value="5.0"/>
+      <origin xyz="0.0 0 0" rpy=" 0 1.5707 1.5707"/>
+      <inertia
+          ixx="0.1" ixy="0" ixz="0"
+          iyy="0.1" iyz="0"
+          izz="0.1"
+      />
+    </inertial>
+    <collision name='rear_left_wheel_collision'>
+      <origin xyz="0 0 0" rpy=" 0 1.5707 1.5707"/>
+      <geometry>
+        <cylinder radius="0.14" length="0.21"/>
+      </geometry>
+    </collision>
+    <visual name='rear_left_wheel_visual'>
+      <origin xyz="0 0 0" rpy=" 0 1.5707 1.5707"/>
+      <geometry>
+        <cylinder radius="0.14" length="0.21"/>
+      </geometry>
+    </visual>
+  </link>
+  <link name='rear_right_wheel'>
+    <pose>0 0 0 0 0 0</pose>
+    <inertial>
+      <mass value="5.0"/>
+      <origin xyz="0.0 0 0" rpy=" 0 1.5707 1.5707"/>
+      <inertia
+          ixx="0.1" ixy="0" ixz="0"
+          iyy="0.1" iyz="0"
+          izz="0.1"
+      />
+    </inertial>
+    <collision name='rear_right_wheel_collision'>
+      <origin xyz="0 0 0" rpy=" 0 1.5707 1.5707"/>
+      <geometry>
+        <cylinder radius="0.14" length="0.21"/>
+      </geometry>
+    </collision>
+    <visual name='rear_right_wheel_visual'>
+      <origin xyz="0 0 0" rpy=" 0 1.5707 1.5707"/>
+      <geometry>
+        <cylinder radius="0.14" length="0.21"/>
+      </geometry>
+    </visual>
+  </link>
+  <joint type="continuous" name="front_left_wheel_hinge">
+    <origin xyz="0.9 0.6 0" rpy="0 0 0"/>
+    <child link="front_left_wheel"/>
+    <parent link="chassis"/>
+    <axis xyz="0 1 0" rpy="0 0 0"/>
+    <limit effort="10000" velocity="1000"/>
+    <dynamics damping="1.0" friction="1.0"/>
+  </joint>
+  <joint type="continuous" name="front_right_wheel_hinge">
+    <origin xyz="0.9 -0.6 0" rpy="0 0 0"/>
+    <child link="front_right_wheel"/>
+    <parent link="chassis"/>
+    <axis xyz="0 1 0" rpy="0 0 0"/>
+    <limit effort="10000" velocity="1000"/>
+    <dynamics damping="1.0" friction="1.0"/>
+  </joint>
+  <joint type="continuous" name="rear_left_wheel_hinge">
+    <origin xyz="-0.9 0.6 0" rpy="0 0 0"/>
+    <child link="rear_left_wheel"/>
+    <parent link="chassis"/>
+    <axis xyz="0 1 0" rpy="0 0 0"/>
+    <limit effort="10000" velocity="1000"/>
+    <dynamics damping="1.0" friction="1.0"/>
+  </joint>
+  <joint type="continuous" name="rear_right_wheel_hinge">
+    <origin xyz="-0.9 -0.6 0" rpy="0 0 0"/>
+    <child link="rear_right_wheel"/>
+    <parent link="chassis"/>
+    <axis xyz="0 1 0" rpy="0 0 0"/>
+    <limit effort="10000" velocity="1000"/>
+    <dynamics damping="1.0" friction="1.0"/>
+  </joint>
+  <link name='camera'>
     <pose>0 0 0 0 0 0</pose>
     <inertial>
@@ -131,5 +255,5 @@
       />
     </inertial>
-    <collision name="collision">
+    <collision name='collision'>
       <origin xyz="0 0 0" rpy=" 0 0 0"/>
       <geometry>
@@ -137,5 +261,5 @@
       </geometry>
     </collision>
-    <visual name="camera_visual">
+    <visual name='camera_visual'>
       <origin xyz="0 0 0" rpy="0 0 0"/>
       <geometry>
@@ -145,5 +269,5 @@
   </link>
   <joint type="fixed" name="camera_joint">
-    <origin xyz="0.2 0 0" rpy="0 0 0"/>
+    <origin xyz="1.0 0 0" rpy="0 0 0"/>
     <child link="camera"/>
     <parent link="chassis"/>
@@ -152,5 +276,5 @@
     <dynamics damping="1.0" friction="1.0"/>
   </joint>
-  <link name="hokuyo">
+  <link name='hokuyo'>
     <pose>0 0 0 0 0 0</pose>
     <inertial>
@@ -163,5 +287,5 @@
       />
     </inertial>
-    <collision name="collision">
+    <collision name='collision'>
       <origin xyz="0 0 0" rpy=" 0 0 0"/>
       <geometry>
@@ -169,5 +293,5 @@
       </geometry>
     </collision>
-    <visual name="hokuyo_visual">
+    <visual name='hokuyo_visual'>
       <origin xyz="0 0 0" rpy="0 0 0"/>
       <geometry>
@@ -177,5 +301,5 @@
   </link>
   <joint type="fixed" name="hokuyo_joint">
-    <origin xyz="0.15 0.0 0.1" rpy="0 0 0"/>
+    <origin xyz="0.8 0.0 0.3" rpy="0 0 0"/>
     <child link="hokuyo"/>
     <parent link="chassis"/>
